File: BaSe_PWR_V3_2.kicad_sch (KiCad schematic)
At the start: 99 parts

Commit message: version with bananapi. Manufactured by jlcpcb and used in hw_rev3b
Parts:
- removed C14: (no value), symbol BackupServer-rescue:C-BackupServer-rescue
- removed Cable_HDD_ENDSW_preconfected1, Conn_Socket_ENDSWHDD1: (no value), symbol Connector:Conn_01x01_Female
- removed FB1, FB9: (no value), symbol Device:Ferrite_Bead_Small
- removed J7: (no value), symbol Connector_Generic:Conn_01x03
- added C14: (no value), symbol BackupServer-rescue:CP-BackupServer-rescue
- added C17, C20: (no value), symbol Device:C_Small
- added D4, D5: (no value), symbol Device:D_Zener
- added D6: (no value), symbol Device:D_Schottky
- added F1: (no value), symbol Device:Fuse
- added FB9, R21, R22, R23, R25, R26, R27: (no value), symbol BackupServer-rescue:R-BackupServer-rescue
- added FL2: (no value), symbol Device:EMI_Filter_LL_1423
- added Q6, Q7: (no value), symbol Transistor_FET:BSS123
- 2k4, R24, R6: SPN (none) -> A129689CT-ND
- C1, C16, C6, C7: SPN (none) -> 399-7845-1-ND
- C12: SPR (none) -> Digikey
- C19: SPN 587-1387-1-ND -> PCE4537CT-ND; Vrated (none) -> 16V
- C24: SPN (none) -> 311-1080-1-ND
- C9: SPN (none) -> 311-1572-1-ND
- D1, D2: SPN (none) -> 1N4148WRHGCT-ND
- D3: SPN 732-9984-1-ND -> 732-9949-1-ND
- Q1, Q5: SPN (none) -> BS170-D75ZCT-ND
- Q2: SPN (none) -> BSS123LT1GOSCT-ND
- Q4: SPN BSC093N04LSGATMA1CT-ND -> BSC093N04LSGATMA1CT-ND
- R1: SPN 696-1369-1-ND -> 696-1369-1-ND
- R10, R11, R12, R13, R9, Ron1: SPN (none) -> 311-47KGRCT-ND
- R19, R5, Rfbt1: SPN (none) -> 311-10.0KHRCT-ND
- R3: SPN (none) -> 311-1.00KHRCT-ND
- U3: SPN (none) -> ADG734BRUZ-REEL7CT-ND
Connections:
- net +12V_HDD: now also FB9.2
- net +12V_HDD_flt: now also FB9.1
- net +3V3: now also R18.1, R21.1, R22.1; no longer M1.17 (3.3V), R20.2, U3.1
- net +3V3_STBY: now also R17.1, R7.2, R27.1; no longer J5.8 (Pin_8)
- net +5V_HDD_flt: no longer J4.8 (Pin_8)
- net 12V_Prot: now also C12.1, D6.1 (K); no longer R18.1
- net 12V_nProt: now also R15.1, D4.1 (K), D6.2 (A), F1.1; no longer C3.1, FL1.4, R18.2
- net 5V_EN: now also R17.2; no longer R17.1
- net DIS_BPi_SPLY: now also R7.1, R25.2; no longer R7.2
- net GND: now also J5.8 (Pin_8), R20.2, C14.2, C17.2, FL2.4, Q6.2 (S), Q7.2 (S), R23.2, R25.1; no longer C12.2, J2.2 (Pin_2), J4.9 (Pin_9), R15.2, R17.2, R20.1, R7.1
- net Taster_0: now also Q6.1 (G); no longer M1.21 (GPIO_13/MISO)
- net Taster_1: now also Q7.1 (G); no longer M1.23 (GPIO_14/SCLK)
- net Vin_Buck: now also C14.1
- net ~{Endswitch_Docked}: now also J4.8 (Pin_8)
- net ~{Endswitch_Undocked}: now also J4.9 (Pin_9)
- net at R3.1, U4.6 (Vss): now also C12.2, D5.1 (K)
- net Vin_Stepper: now reaches C18.1, FB2.2, SCT1.16 (VMOT)
- net MS1: now reaches R9.1, SCT1.2 (MS1)
- net MS1: now also R18.2
- net MS2: now reaches R10.1, SCT1.3 (MS2)
- net MS2: now also R21.2
- net MS3: now reaches R11.1, SCT1.4 (ME3)
- net MS3: now also R22.2
- net at J2.1 (Pin_1): now also C20.2, FL2.1; no longer C12.1
- net at Q4.1 (S), Q4.2 (S), Q4.3 (S): now also C17.1, FL2.3
- net EN_attiny_link: now reaches M1.22 (GPIO_6)
- net EN_attiny_link: now also R20.1, U3.1
- net Dis_PWM_attiny renamed Version
- net Version: now also R23.1, R26.2
- net LTC4359_~{SHDN}: no longer names the net of U4.5 (~{SHDN})
- net LTC4359_~{SHDN}: now also R15.2; no longer R15.1
- net ~{LTC4359_SHDN}: no longer names the net of U5.6 (PB5)
- new net: C3.1, F1.2, FL1.4
- new net: D4.2 (A), D5.2 (A)
- new net: C20.1, FL2.2, J2.2 (Pin_2)
- new net: R26.1, R27.2
- new net ~{Taster_0}: M1.21 (GPIO_13/MISO), Q6.3 (D)
- new net ~{Taster_1}: M1.23 (GPIO_14/SCLK), Q7.3 (D)
- no-connect marks 21 -> 20
Other:
- note added: "(R25 fitted) if DIS_BPi_SLPY = HiZ: Q2 Opens Q4 conducts 5V is passed to BPi"
- note added: "0R instead of Ferrite. Ferrite prevents the HDD from starting up"
- note added: "fsw = 500kHz"
- note added: "polarity checked"
- moved on the sheet: C1, C15, C18, C19, C5, Cable_BPi_SPLY_preconfected1, Cable_BPi_SPLY_preconfected2, Conn_Socket_BPi_SPLY1, Conn_Socket_BPi_SPLY_atJ5, FB10, FB2, FB7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
