File: BaSe_PWR_V3_3.kicad_sch (KiCad schematic)
At the start: 110 parts

Commit message: replace analog switches by cheaper ones
Parts:
- removed FB9, R23, R27: (no value), symbol BackupServer-rescue:R-BackupServer-rescue
- removed U3: (no value), symbol Analog_Switch:ADG734
- added 2k1, R11: (no value), symbol BackupServer-rescue:R-BackupServer-rescue
- added C11, C15: (no value), symbol BackupServer-rescue:C-BackupServer-rescue
- added FB7: (no value), symbol Device:Ferrite_Bead_Small
- added U3, U4, U5: (no value), symbol Analog_Switch:NC7SB3157P6X
- 2k2: renamed from R6; SPN A129689CT-ND -> (none)
- 2k5: renamed from R24; SPN A129689CT-ND -> (none)
- 2k7: renamed from 2k4; SPN A129689CT-ND -> (none)
- C10: renamed from C7; SPN 399-7845-1-ND -> (none)
- C12: renamed from C6; SPN 399-7845-1-ND -> (none)
- C17: renamed from C9; SPN 311-1572-1-ND -> (none)
- C19: renamed from C24; SPN 311-1080-1-ND -> (none)
- C3: renamed from C16; SPN 399-7845-1-ND -> (none)
- C8: renamed from C1; SPN 399-7845-1-ND -> (none)
- D4: renamed from D6; SPN SK64L-TPMSCT-ND -> (none)
- D5: renamed from D1; SPN 1N4148WRHGCT-ND -> (none)
- D6: renamed from D2; SPN 1N4148WRHGCT-ND -> (none)
- Q1: renamed from Q6; SPN BSS123LT1GOSCT-ND -> (none)
- Q2: renamed from Q7; SPN BSS123LT1GOSCT-ND -> (none)
- Q4: renamed from Q1; SPN BS170-D75ZCT-ND -> (none)
- Q5: renamed from Q2; SPN BSS123LT1GOSCT-ND -> (none)
- Q6: renamed from Q4; SPN BSC093N04LSGATMA1CT-ND -> BSC093N04LSGATMA1CT-ND
- Q7: renamed from Q5; SPN BS170-D75ZCT-ND -> (none)
- R10: renamed from R13; SPN 311-47KGRCT-ND -> (none)
- R12: renamed from R1; Digikey 696-1369-1-ND‎ -> 696-1369-1-ND‎ (END OF LIFE); MPN CSR1206-0R001F1 -> CSR1206-0R001F1 (END OF LIFE); SPN 696-1369-1-ND -> 696-1369-1-ND (END OF LIFE)
- R15: renamed from R5; SPN 311-10.0KHRCT-ND -> (none)
- R16: renamed from R19; SPN 311-10.0KHRCT-ND -> (none)
- R2: renamed from R9; SPN 311-47KGRCT-ND -> (none)
- R20: renamed from Rfbt1; SPN 311-10.0KHRCT-ND -> (none)
- R4: renamed from R10; SPN 311-47KGRCT-ND -> (none)
- R6: renamed from R11; SPN 311-47KGRCT-ND -> (none)
- R7: renamed from R12; SPN 311-47KGRCT-ND -> (none)
- R9: renamed from R3; SPN 311-1.00KHRCT-ND -> (none)
- Rfbt2: renamed from Ron1; SPN 311-47KGRCT-ND -> (none)
- renumbered R8 to 2k3, R7 to 2k4, 2k3 to 2k6, C2 to C1, C14 to C13, C8 to C14, C10 to C16, C13 to C18, C3 to C2, C11 to C20, C4 to C21, C17 to C22, C20 to C23, C18 to C4, C19 to C5, C12 to C6, C15 to C7, C5 to C9, Cable_HDD_ENDSW_preconfected2 to Cable_HDD_ENDSW_preconfected1, Conn_Socket_BPi_SPLY_atJ5 to Conn_Socket_BPi_SPLY_atJ1, D3 to D1, D4 to D2, D5 to D3, FB2 to FB1, FB3 to FB2, FB4 to FB3, FB5 to FB4, FB6 to FB5, FB7 to FB6, FB10 to FB8, J6 to J2, J5 to J4, J4 to J5, J2 to J6, R18 to R1, R2 to R13, R4 to R14, R20 to R17, R14 to R18, R26 to R19, Rfbb1 to R21, R25 to R22, R16 to R23, R21 to R3, R22 to R5, R15 to R8, R17 to Rfbt1, U4 to U1, U1 to U2, U5 to U6, U2 to U8
Connections:
- net +12V_HDD: now also FB7.2
- net +12V_HDD_flt: now also FB7.1
- net +3V3: now also R17.1, R19.1, U5.6
- net +3V3_STBY: now also C11.1, C15.1, U3.5 (V+), U4.5 (V+), U5.5 (V+)
- net 12V_nProt: now also D1.1 (A1)
- net DC_IN+: no longer D1.1 (A1)
- net DC_IN-: no longer D1.2 (A2)
- net EN_attiny_link: no longer R17.1
- net GND: now also D1.2 (A2), C11.2, C15.2, U3.2 (GND), U4.2 (GND), U5.2 (GND), U5.3
- net RxD_BPi: now also R11.1, U4.4; no longer M1.10 (GPIO_16/RxD)
- net RxD_attiny: now also U3.3
- net TxD_BPi: now also U3.4
- net TxD_attiny: now also U5.1
- net TxD_attiny_prot: now also U4.3, U5.4
- net attiny_program_~{communicate}: now also U3.6, U4.6
- net attiny_~{reset}: now also U4.1
- net BPi_Heartbeat_prot: now reaches U6.6 (PB5)
- net BPi_Heartbeat_prot: now also 2k1.2
- net at R15.2, R16.2: now also U3.1
- net BPi_Heartbeat: now reaches M1.24 (GPIO_10/CS0)
- net BPi_Heartbeat: now also 2k1.1
- net Version renamed +3V3_Sense
- new net RxD_BPi_prot: M1.10 (GPIO_16/RxD), R11.2
- no-connect marks 20 -> 19
Other:
- note added: "(Reverse Polarity Prot.)"
- note added: "BCU <> SBU Communication and Programming Switch"
- note added: "BPi Power Switch"
- note added: "Backup Control Unit (BCU)"
- note added: "DC Voltage regulators"
- note added: "HDD Power Switch"
- note added: "HMI Connector"
- note added: "Ideal Diode"
- note added: "Input Current Measurement Unit"
- note added: "Signal added in V3_3"
- note added: "Standby Unit (SBU)"
- note added: "Stepper Driver and Connector"
- note added: "deprectated"
- note added: "moved here in V3_3"
- note removed: "+3V3_STBY is generated by a linear regulator, therefore it should have less ripple than +3V3 (from rpi)"
- note removed: "0R instead of Ferrite. Ferrite prevents the HDD from starting up"
- title: BaSe_PWR_V3_1 -> BaSe_PWR_V3_3
- moved on the sheet: 2k2, 2k3, 2k5, 2k6, 2k7, C1, C10, C12, C2, C8, C9, Cable_HDD_ENDSW_preconfected1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
